File: ROMSIMM.kicad_pcb (KiCad board)
At the start: 4 copper layers, 97.8 x 25 mm, 40 parts, among them J1 ROM, SW1 ROM Sel., U1 MX29LV640, U10 74AHC245, U11 XC6206P332MR, U12 74LVC1G02GW, U2 MX29LV640, U3 74AHC245, U4 74AHC245, U5 74AHC245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

Commit message: Add new GW logotype
Parts:
- added G***: LOGO, LOGO, B.Cu at (99.6, 113.4)
- added G***: LOGO, LOGO, B.Cu at (144.7, 113.5)
Routing:
- net +3V3: track 58.2 -> 76.2 mm, vias 74 -> 76
- net /RA21: track 29.5 -> 28.2 mm
- net GND: track 84.1 -> 82.9 mm, vias 152 -> 144
- net /RA22sw: track 80.2 -> 81.2 mm
- net /R~{OE}: track 80.1 -> 80.9 mm
Other:
- board text removed: "4402C"
- board text removed: "8 MB ROM SIMM"
- board text removed: "GW"
- board text removed: "Garrett’s Workshop"
- board text removed: "for Mac II and SE/30"
