File: MacIIROMSIMM.kicad_pcb (KiCad board)
At the start: 4 copper layers, 97.8 x 25 mm, 42 parts, among them J1 ROM, SW1 ROM Sel., U1 MX29LV640, U10 74AHC245, U11 XC6206P332MR, U12 74LVC1G02GW, U2 MX29LV640, U3 74AHC245, U4 74AHC245, U5 74AHC245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

Commit message: idk build?
Parts:
- moved G*** 0.47 mm to (100.0, 113.7)
- turned U12 to 0 degrees

Commit message: Build and changed text to 4402B
Routing:
- net +3V3: track 76.2 -> 77.3 mm, vias 76 -> 75
- net GND: track 82.9 -> 83.8 mm
- net /RA22: track 31.2 -> 31.9 mm

Commit message: RC
Other:
- rule pad_to_mask_clearance: 0.075 -> 0.0762
- rule solder_mask_min_width: 0.1 -> 0.127
- board text added: "JLCJLCJLCJLC"

Commit message: RC
Parts:
- U10, U3, U4, U5, U6, U7, U9: value 74AHC245 -> 74LVC245APW
Routing:
- net +5V: track 166.3 -> 164.0 mm
