File: MacIIROMSIMM.kicad_sch (KiCad schematic)
At the start: 40 parts, among them J1 ROM, SW1 ROM Sel., U1 MX29LV640, U10 74AHC245, U11 XC6206P332MR, U12 74LVC1G02GW, U2 MX29LV640, U3 74AHC245, U4 74AHC245, U5 74AHC245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

Commit message: Build and changed text to 4402B
Parts:
- H1, H2, H3, H4: symbol Mechanical:MountingHole_Pad -> Mechanical:MountingHole
Connections:
- net GND: no longer H1.1, H2.1, H3.1, H4.1

Commit message: RC
Parts:
- SW1: LCSC Part C319052 -> C319051
- U1, U2: LCSC Part C117907 -> C30076
- U10, U3, U4, U5, U6, U7, U9: value 74AHC245 -> 74LVC245APW; LCSC Part C132987 -> C6082
